File: electronics/view_screen/view_screen.kicad_sch (KiCad schematic)
At the start: 17 parts, among them J2 GC9A01, J6 LCD - FPC, Q1 2N7002

Commit message: Cleaned up electronics
Other:
- note added: "Additional Design by Seedlabs"
- note added: "LCD connector"
- note added: "Original Design by Scott Bezek"
- company: (none) -> Seedlabs
- title: (none) -> SmartKnob DevKit Screen
- moved on the sheet: C1, C2, H1, J2, J6, Q1, R1, R2, R3, TP1, TP2, TP3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
